Commit message: Add files via upload
Added hole to front of robot
Added arm to robot
Made an airport runway in gazebo
spawn_garbage.py spawns up to 5 garbages at a time

File: urdf/arm.urdf (robot description, URDF)
Before this commit: robot arm6_joint, 0 links, 0 joints
Links:
- added link arm1_p_link; collision cylinder length=0.1 radius=0.1; visual cylinder length=0.1 radius=0.1
- added link arm1_r_link; collision cylinder length=0.1 radius=0.1; visual cylinder length=0.1 radius=0.1
- added link arm2_link; collision box size=0.2 0.2 0.1; collision box size=0.2 0.2 0.1
- added link arm3_link; collision box size=0.2 0.2 0.1; collision cylinder length=0.5 radius=0.1
- added link arm4_link; collision cylinder length=0.1 radius=0.1; collision cylinder length=0.5 radius=0.08
- added link base_link; collision box size=0.2 1 0.1; visual box size=0.2 1 0.1
- added link tool_link
Joints:
- added joint arm1_p_joint: type prismatic, parent base_link, child arm1_p_link, origin xyz=0 0 0.1 rpy=0 0 0, axis 0 1 0, limit lower=0.4 upper=-0.4 effort=100 velocity=0.1
- added joint arm1_r_joint: type revolute, parent arm1_p_link, child arm1_r_link, origin xyz=0 0 0.1 rpy=0 0 0, axis 0 0 1, limit lower=6.28318530718 upper=-6.28318530718 effort=100 velocity=0.1
- added joint arm2_joint: type revolute, parent arm1_r_link, child arm2_link, origin xyz=0 -0.2 -0 rpy=0 0 0, axis 0 1 0, limit lower=6.28318530718 upper=-6.28318530718 effort=100 velocity=0.1
- added joint arm3_joint: type revolute, parent arm2_link, child arm3_link, origin xyz=0 0.2 0.6 rpy=0 0 0, axis 0 1 0, limit lower=6.28318530718 upper=-6.28318530718 effort=100 velocity=0.1
- added joint arm4_joint: type prismatic, parent arm3_link, child arm4_link, origin xyz=0 0 0.3 rpy=0 0 0, axis 0 0 1, limit lower=0 upper=0.5 effort=100 velocity=0.1
- added joint tool_joint: type fixed, parent arm4_link, child tool_link, origin xyz=0 0 0.3 rpy=0 0 0

File: urdf/irwb.xacro (robot description, xacro)
@@ -6,8 +6,12 @@
 <!-- ########################################### -->
 <robot name="runway_bot" xmlns:xacro="http://www.ros.org/wiki/xacro">
+  <xacro:include filename="$(find irwb_robot_pkg)/urdf/arm.xacro"/>
   <!-- Body dimensions -->
   <xacro:property name="body_link_x_dim" value="2"/>
   <xacro:property name="body_link_y_dim" value="1"/>
   <xacro:property name="body_link_z_dim" value="0.7"/>
+  <xacro:property name="body_inner_x" value="0.8"/>
+  <xacro:property name="body_inner_y" value="0.8"/>
+  <xacro:property name="body_inner_z" value="0.6"/>
   <!-- Wheel dimensions -->
   <xacro:property name="wheel_link_radius" value="0.2"/>
@@ -16,5 +20,5 @@
   <!-- Material density -->
   <xacro:property name="body_density" value="2710"/>
-  <xacro:property name="wheel_density" value="2710"/>
+  <xacro:property name="wheel_density" value="1500"/>
   <!-- Pi const -->
   <xacro:property name="pi_const" value="3.141592652589"/>
@@ -46,16 +50,78 @@
     <child link="body_link"/>
   </joint>
-  <!--### Body link of iRWB ###-->
+  <!--####################################-->
+  <!--# body_link with hole in the front #-->
+  <!--####################################-->
   <link name="body_link">
     <visual>
-      <origin rpy="0 0 0" xyz="0 0 0"/>
-      <geometry>
-        <box size="${body_link_x_dim} ${body_link_y_dim} ${body_link_z_dim}"/>
-      </geometry>
-    </visual>
-    <collision>
-      <origin rpy="0 0 0" xyz="0 0 0"/>
-      <geometry>
-        <box size="${body_link_x_dim} ${body_link_y_dim} ${body_link_z_dim}"/>
+      <origin rpy="0 0 0" xyz="${-1 * body_link_x_dim / 4} 0 0"/>
+      <geometry>
+        <box size="${body_link_x_dim / 2} ${body_link_y_dim} ${body_link_z_dim}"/>       <!-- Solid back part -->
+      </geometry>
+    </visual>
+    <visual>
+      <origin rpy="0 0 0" xyz="${(body_link_x_dim/2 - body_inner_x)/4.0} 0 0"/>       <!-- Shaded area 1 -->
+      <geometry>
+        <box size="0.1 ${body_inner_y} ${body_link_z_dim}"/>
+      </geometry>
+    </visual>
+    <visual>
+      <origin rpy="0 0 0" xyz="${(body_link_x_dim/2 - body_inner_x)/4 + 0.9} 0 0"/>  <!-- Shaded area 2 -->
+      <geometry>
+        <box size="0.1 ${body_inner_y} ${body_link_z_dim}"/>
+      </geometry>
+    </visual>
+    <visual>
+      <origin rpy="0 0 0" xyz="${body_link_x_dim / 4} ${(body_link_y_dim - 0.1)/ 2} 0"/>  <!-- Unshaded area 1 -->
+      <geometry>
+        <box size="${body_inner_x + 0.2} 0.1 ${body_link_z_dim}"/>
+      </geometry>
+    </visual>
+    <visual>
+      <origin rpy="0 0 0" xyz="${body_link_x_dim / 4} ${-1 * (body_link_y_dim - 0.1)/ 2} 0"/> <!-- Unshaded area 2 -->
+      <geometry>
+        <box size="${body_inner_x + 0.2} 0.1 ${body_link_z_dim}"/>
+      </geometry>
+    </visual>
+    <visual>
+      <origin rpy="0 0 0" xyz="${body_link_x_dim / 4} 0 ${-1 * (body_link_z_dim - 0.1)/2}"/> <!-- Base of hole -->
+      <geometry>
+        <box size="${body_inner_x} ${body_inner_y} 0.1"/>
+      </geometry>
+    </visual>
+    <collision>
+      <origin rpy="0 0 0" xyz="${-1 * body_link_x_dim / 4} 0 0"/>
+      <geometry>
+        <box size="${body_link_x_dim / 2} ${body_link_y_dim} ${body_link_z_dim}"/>
+      </geometry>
+    </collision>
+    <collision>
+      <origin rpy="0 0 0" xyz="${(body_link_x_dim/2 - body_inner_x)/4.0} 0 0"/>
+      <geometry>
+        <box size="0.1 ${body_inner_y} ${body_link_z_dim}"/>
+      </geometry>
+    </collision>
+    <collision>
+      <origin rpy="0 0 0" xyz="${(body_link_x_dim/2 - body_inner_x)/4 + 0.9} 0 0"/>
+      <geometry>
+        <box size="0.1 ${body_inner_y} ${body_link_z_dim}"/>
+      </geometry>
+    </collision>
+    <collision>
+      <origin rpy="0 0 0" xyz="${body_link_x_dim / 4} ${(body_link_y_dim - 0.1)/ 2} 0"/>
+      <geometry>
+        <box size="${body_inner_x + 0.2} 0.1 ${body_link_z_dim}"/>
+      </geometry>
+    </collision>
+    <collision>
+      <origin rpy="0 0 0" xyz="${body_link_x_dim / 4} ${-1 * (body_link_y_dim - 0.1)/ 2} 0"/>
+      <geometry>
+        <box size="${body_inner_x + 0.2} 0.1 ${body_link_z_dim}"/>
+      </geometry>
+    </collision>
+    <collision>
+      <origin rpy="0 0 0" xyz="${body_link_x_dim / 4} 0 ${-1 * (body_link_z_dim - 0.1)/2}"/>
+      <geometry>
+        <box size="${body_inner_x} ${body_inner_y} 0.1"/>
       </geometry>
     </collision>
@@ -73,4 +139,7 @@
     </inertial>
   </link>
+  <!--####################################-->
+  <!--#         end of body_link         #-->
+  <!--####################################-->
  <!--# Joint from iRWB to wheel 1 #-->
  <joint name="wheel1_joint" type="continuous">
@@ -185,3 +254,9 @@
     <xacro:inertia_wheel/>
   </link>
+  <!-- Fixed Joint from arm to body -->
+  <joint name="arm_mount_joint" type="fixed">
+    <parent link="body_link"/>
+    <child link="base_link"/>
+    <origin rpy="0 0 0" xyz="0 0 0.4"/>
+  </joint>
 </robot>
