Commit message: Add files via upload

File: urdf/arm.xacro (robot description, xacro)
@@ -1,51 +1,100 @@
 <?xml version="1.0"?>
 <robot name="arm_robot" xmlns:xacro="http://www.ros.org/wiki/xacro">
-  <!-- Properties -->
-  <xacro:property name="density" value="2700"/>  <!-- Density in kg/m^3 -->
-  <!-- Macro for calculating inertia for a box -->
-  <xacro:macro name="inertia_box" params="mass x y z">
-    <inertial>
-      <mass value="${mass}"/>
-      <origin rpy="0 0 0" xyz="0 0 0"/>
-      <inertia
-        ixx="${mass * (y*y + z*z) / 12.0}"
-        iyy="${mass * (x*x + z*z) / 12.0}"
-        izz="${mass * (x*x + y*y) / 12.0}"
-        ixy="0.0"
-        ixz="0.0"
-        iyz="0.0" />
-    </inertial>
+  <!-- Constants -->
+  <xacro:property name="density" value="2710"/> <!-- Aluminum density kg/m³ -->
+  <xacro:property name="pi" value="3.1415926535897931"/>
+  <!-- Materials -->
+  <material name="aluminum">
+    <color rgba="0.7 0.7 0.7 1"/>
+  </material>
+  <material name="gripper_color">
+    <color rgba="0.9 0.9 0.9 1"/>
+  </material>
+  <!-- Generic Cylinder Macro -->
+  <xacro:macro name="cylinder_link" params="name radius length origin_xyz origin_rpy">
+    <link name="${name}">
+      <xacro:property name="mass" value="${density * pi * radius*radius * length}"/>
+      <visual>
+        <origin rpy="${origin_rpy}" xyz="${origin_xyz}"/>
+        <geometry>
+          <cylinder radius="${radius}" length="${length}"/>
+        </geometry>
+        <material name="aluminum"/>
+      </visual>
+      <collision>
+        <origin rpy="${origin_rpy}" xyz="${origin_xyz}"/>
+        <geometry>
+          <cylinder radius="${radius}" length="${length}"/>
+        </geometry>
+      </collision>
+      <inertial>
+        <origin rpy="${origin_rpy}" xyz="${origin_xyz}"/>
+        <mass value="${mass}"/>
+        <inertia
+          ixx="${(mass/12) * (3*radius*radius + length*length)}"
+          ixy="0"
+          ixz="0"
+          iyy="${(mass/12) * (3*radius*radius + length*length)}"
+          iyz="0"
+          izz="${0.5 * mass * radius*radius}"/>
+      </inertial>
+    </link>
   </xacro:macro>
-  <!-- Macro for calculating inertia for a cylinder -->
-  <xacro:macro name="inertia_cylinder" params="mass radius length">
-    <inertial>
-      <mass value="${mass}"/>
-      <origin rpy="0 0 0" xyz="0 0 0"/>
-      <inertia
-        ixx="${mass * (3*radius*radius + length*length) / 12.0}"
-        iyy="${mass * (3*radius*radius + length*length) / 12.0}"
-        izz="${mass * radius*radius / 2.0}"
-        ixy="0.0"
-        ixz="0.0"
-        iyz="0.0" />
-    </inertial>
+  <!-- Generic Box Macro -->
+  <xacro:macro name="box_link" params="name size_x size_y size_z origin_xyz origin_rpy">
+    <link name="${name}">
+      <xacro:property name="mass" value="${density * size_x * size_y * size_z}"/>
+      <visual>
+        <origin rpy="${origin_rpy}" xyz="${origin_xyz}"/>
+        <geometry>
+          <box size="${size_x} ${size_y} ${size_z}"/>
+        </geometry>
+        <material name="aluminum"/>
+      </visual>
+      <collision>
+        <origin rpy="${origin_rpy}" xyz="${origin_xyz}"/>
+        <geometry>
+          <box size="${size_x} ${size_y} ${size_z}"/>
+        </geometry>
+      </collision>
+      <inertial>
+        <origin rpy="${origin_rpy}" xxyz="${origin_xyz}"/>
+        <mass value="${mass}"/>
+        <inertia
+          ixx="${(mass/12) * (size_y*size_y + size_z*size_z)}"
+          ixy="0"
+          ixz="0"
+          iyy="${(mass/12) * (size_x*size_x + size_z*size_z)}"
+          iyz="0"
+          izz="${(mass/12) * (size_x*size_x + size_y*size_y)}"/>
+      </inertial>
+    </link>
   </xacro:macro>
-  <!-- Base Link -->
-  <link name="base_link">
-    <visual>
-      <origin rpy="0 0 0" xyz="0 0 0"/>
-      <geometry>
-        <box size="0.2 1 0.1"/>
-      </geometry>
-    </visual>
-    <collision>
-      <origin rpy="0 0 0" xyz="0 0 0"/>
-      <geometry>
-        <box size="0.2 1 0.1"/>
-      </geometry>
-    </collision>
-    <xacro:inertia_box mass="${density * 0.2 * 1 * 0.1}" x="0.2" y="1" z="0.1"/>
-  </link>
-  <!-- Prismatic Joint -->
+  <!-- Arm Link Components -->
+  <xacro:box_link name="base_link"
+    size_x="0.2" size_y="1" size_z="0.1"
+    origin_xyz="0 0 0" origin_rpy="0 0 0"/>
+  <xacro:cylinder_link name="arm1_p_link"
+    radius="0.1" length="0.1"
+    origin_xyz="0 0 0" origin_rpy="0 0 0"/>
+  <xacro:cylinder_link name="arm1_r_link"
+    radius="0.1" length="0.1"
+    origin_xyz="0 0 0" origin_rpy="0 0 0"/>
+  <xacro:cylinder_link name="arm2_link"
+    radius="0.1" length="0.5"
+    origin_xyz="0 0 ${(0.5-0.1)/2}" origin_rpy="0 0 0"/>
+  <xacro:cylinder_link name="arm3_link"
+    radius="0.1" length="0.5"
+    origin_xyz="0 0 ${(0.5-0.1)/2}" origin_rpy="0 0 0"/>
+  <xacro:cylinder_link name="arm4_link"
+    radius="0.08" length="0.5"
+    origin_xyz="0 0 ${(0.5-0.1)/2}" origin_rpy="0 0 0"/>
+  <xacro:cylinder_link name="arm5_link"
+    radius="0.1" length="0.02"
+    origin_xyz="0 0 0" origin_rpy="0 0 0"/>
+  <xacro:box_link name="arm6_link"
+    size_x="0.02" size_y="0.2" size_z="0.02"
+    origin_xyz="0 0 0" origin_rpy="0 0 0"/>
+  <!-- Arm Joints -->
   <joint name="arm1_p_joint" type="prismatic">
     <parent link="base_link"/>
@@ -53,23 +102,6 @@
     <origin rpy="0 0 0" xyz="0 0 0.1"/>
     <axis xyz="0 1 0"/>
-    <limit lower="-0.4" upper="0.4" effort="50" velocity="0.2"/>
+    <limit lower="-0.4" upper="0.4" effort="100" velocity="0.1"/>
   </joint>
-  <!-- First Prismatic Link -->
-  <link name="arm1_p_link">
-    <visual>
-      <origin rpy="0 0 0" xyz="0 0 0"/>
-      <geometry>
-        <cylinder radius="0.1" length="0.1"/>
-      </geometry>
-    </visual>
-    <collision>
-      <origin rpy="0 0 0" xyz="0 0 0"/>
-      <geometry>
-        <cylinder radius="0.1" length="0.1"/>
-      </geometry>
-    </collision>
-    <xacro:inertia_cylinder mass="${density * 3.14 * 0.1 * 0.1 * 0.1}" radius="0.1" length="0.1"/>
-  </link>
-  <!-- Revolute Joint -->
   <joint name="arm1_r_joint" type="revolute">
     <parent link="arm1_p_link"/>
@@ -77,194 +109,61 @@
     <origin rpy="0 0 0" xyz="0 0 0.1"/>
     <axis xyz="0 0 1"/>
-    <limit lower="-3.14" upper="3.14" effort="50" velocity="1.0"/>
+    <limit lower="-1.57" upper="1.57" effort="100" velocity="0.1"/>
   </joint>
-  <!-- First Revolute Link -->
-  <link name="arm1_r_link">
-    <visual>
-      <origin rpy="0 0 0" xyz="0 0 0"/>
-      <geometry>
-        <cylinder radius="0.1" length="0.1"/>
-      </geometry>
-    </visual>
-    <collision>
-      <origin rpy="0 0 0" xyz="0 0 0"/>
-      <geometry>
-        <cylinder radius="0.1" length="0.1"/>
-      </geometry>
-    </collision>
-    <xacro:inertia_cylinder mass="${density * 3.14 * 0.1 * 0.1 * 0.1}" radius="0.1" length="0.1"/>
-  </link>
-  <!-- Revolute Joint -->
   <joint name="arm2_joint" type="revolute">
     <parent link="arm1_r_link"/>
     <child link="arm2_link"/>
-    <origin rpy="0 0 0" xyz="0 -0.2 0"/>
+    <origin rpy="0 0 0" xyz="0 -0.2 -0"/>
     <axis xyz="0 1 0"/>
-    <limit lower="-3.14" upper="3.14" effort="50" velocity="1.0"/>
+    <limit lower="-1.68" upper="2.01" effort="100" velocity="0.1"/>
   </joint>
-  <!-- Second Link -->
-  <link name="arm2_link">
-    <visual>
-      <origin rpy="0 0 0" xyz="0 0 0"/>
-      <geometry>
-        <box size="0.2 0.2 0.1"/>
-      </geometry>
-    </visual>
-    <visual>
-      <origin rpy="0 0 0" xyz="0 0 0.3"/>
-      <geometry>
-        <cylinder radius="0.1" length="0.5"/>
-      </geometry>
-    </visual>
-    <visual>
-      <origin rpy="0 0 0" xyz="0 0 0.6"/>
-      <geometry>
-        <box size="0.2 0.2 0.1"/>
-      </geometry>
-    </visual>
-    <collision>
-      <origin rpy="0 0 0" xyz="0 0 0"/>
-      <geometry>
-        <box size="0.2 0.2 0.1"/>
-      </geometry>
-    </collision>
-    <collision>
-      <origin rpy="0 0 0" xyz="0 0 0.3"/>
-      <geometry>
-        <cylinder radius="0.1" length="0.5"/>
-      </geometry>
-    </collision>
-    <collision>
-      <origin rpy="0 0 0" xyz="0 0 0.6"/>
-      <geometry>
-        <box size="0.2 0.2 0.1"/>
-      </geometry>
-    </collision>
-    <xacro:inertia_box mass="${density * 0.2 * 0.2 * 0.1}" x="0.2" y="0.2" z="0.1"/>
-  </link>
-  <!-- Revolute Joint -->
   <joint name="arm3_joint" type="revolute">
     <parent link="arm2_link"/>
     <child link="arm3_link"/>
-    <origin rpy="0 0 0" xyz="0 0.2 0.6"/>
+    <origin rpy="0 0 0" xyz="0 0.2 0.4"/>
     <axis xyz="0 1 0"/>
-    <limit lower="-3.14" upper="3.14" effort="50" velocity="1.0"/>
+    <limit lower="-2.80" upper="2.80" effort="100" velocity="0.1"/>
   </joint>
-  <!-- Third Link -->
-  <link name="arm3_link">
-    <visual>
-      <origin rpy="0 0 0" xyz="0 0 0"/>
-      <geometry>
-        <box size="0.2 0.2 0.1"/>
-      </geometry>
-    </visual>
-    <visual>
-      <origin rpy="0 0 0" xyz="0 0 0.3"/>
-      <geometry>
-        <cylinder radius="0.1" length="0.5"/>
-      </geometry>
-    </visual>
-    <collision>
-      <origin rpy="0 0 0" xyz="0 0 0"/>
-      <geometry>
-        <box size="0.2 0.2 0.1"/>
-      </geometry>
-    </collision>
-    <collision>
-      <origin rpy="0 0 0" xyz="0 0 0.3"/>
-      <geometry>
-        <cylinder radius="0.1" length="0.5"/>
-      </geometry>
-    </collision>
-    <xacro:inertia_box mass="${density * 0.2 * 0.2 * 0.1}" x="0.2" y="0.2" z="0.1"/>
-  </link>
-  <!-- Prismatic Joint -->
   <joint name="arm4_joint" type="prismatic">
     <parent link="arm3_link"/>
     <child link="arm4_link"/>
-    <origin rpy="0 0 0" xyz="0 0 0.3"/>
+    <origin rpy="0 0 0" xyz="0 0 0"/>
     <axis xyz="0 0 1"/>
-    <limit lower="0" upper="0.5" effort="50" velocity="0.2"/>
+    <limit lower="0" upper="0.5" effort="100" velocity="0.1"/>
   </joint>
-  <!-- Fourth Link -->
-  <link name="arm4_link">
-    <visual>
-      <origin rpy="0 0 0" xyz="0 0 0"/>
-      <geometry>
-        <cylinder radius="0.08" length="0.5"/>
-      </geometry>
-    </visual>
-    <visual>
-      <origin rpy="0 0 0" xyz="0 0 0.3"/>
-      <geometry>
-        <cylinder length="0.1" radius="0.1" />
-      </geometry>
-    </visual>
-    <collision>
-      <origin rpy="0 0 0" xyz="0 0 0"/>
-      <geometry>
-        <cylinder radius="0.08" length="0.5"/>
-      </geometry>
-    </collision>
-    <collision>
-      <origin rpy="0 0 0" xyz="0 0 0.3"/>
-      <geometry>
-        <cylinder length="0.1" radius="0.1" />
-      </geometry>
-    </collision>
-    <xacro:inertia_cylinder mass="${density * 3.14 * 0.08 * 0.08 * 0.5}" radius="0.08" length="0.5"/>
-  </link>
-  <!-- Fixed Joint for Tool -->
-  <joint name="tool_joint" type="fixed">
+  <joint name="arm5_joint" type="revolute">
     <parent link="arm4_link"/>
-    <child link="tool_link"/>
-    <origin rpy="0 0 0" xyz="0 0 0.3"/>
+    <child link="arm5_link"/>
+    <origin rpy="0 0 0" xyz="0 0 0.45"/>
+    <axis xyz="0 0 1"/>
+    <limit lower="-2.80" upper="2.80" effort="100" velocity="0.1"/>
   </joint>
-  <link name="tool_link"/>
-  <!-- Transmissions -->
-  <transmission name="trans_arm1_p_joint">
-    <type>transmission_interface/SimpleTransmission</type>
-    <joint name="arm1_p_joint">
-      <hardwareInterface>hardware_interface/EffortJointInterface</hardwareInterface>
-    </joint>
-    <actuator name="actuator_arm1_p">
-      <mechanicalReduction>1</mechanicalReduction>
-    </actuator>
-  </transmission>
-  <transmission name="trans_arm1_r_joint">
-    <type>transmission_interface/SimpleTransmission</type>
-    <joint name="arm1_r_joint">
-      <hardwareInterface>hardware_interface/EffortJointInterface</hardwareInterface>
-    </joint>
-    <actuator name="actuator_arm1_r">
-      <mechanicalReduction>1</mechanicalReduction>
-    </actuator>
-  </transmission>
-  <transmission name="trans_arm2_joint">
-    <type>transmission_interface/SimpleTransmission</type>
-    <joint name="arm2_joint">
-      <hardwareInterface>hardware_interface/EffortJointInterface</hardwareInterface>
-    </joint>
-    <actuator name="actuator_arm2">
-      <mechanicalReduction>1</mechanicalReduction>
-    </actuator>
-  </transmission>
-  <transmission name="trans_arm3_joint">
-    <type>transmission_interface/SimpleTransmission</type>
-    <joint name="arm3_joint">
-      <hardwareInterface>hardware_interface/EffortJointInterface</hardwareInterface>
-    </joint>
-    <actuator name="actuator_arm3">
-      <mechanicalReduction>1</mechanicalReduction>
-    </actuator>
-  </transmission>
-  <transmission name="trans_arm4_joint">
-    <type>transmission_interface/SimpleTransmission</type>
-    <joint name="arm4_joint">
-      <hardwareInterface>hardware_interface/EffortJointInterface</hardwareInterface>
-    </joint>
-    <actuator name="actuator_arm4">
-      <mechanicalReduction>1</mechanicalReduction>
-    </actuator>
-  </transmission>
+  <joint name="arm6_joint" type="fixed">
+    <parent link="arm5_link"/>
+    <child link="arm6_link"/>
+    <origin rpy="0 0 0" xyz="0 0 0.02"/>
+  </joint>
+  <!-- Gripper Components -->
+  <xacro:box_link name="gripper_left"
+    size_x="0.02" size_y="0.02" size_z="0.1"
+    origin_xyz="0 0 0" origin_rpy="0 0 0"/>
+  <xacro:box_link name="gripper_right"
+    size_x="0.02" size_y="0.02" size_z="0.1"
+    origin_xyz="0 0 0" origin_rpy="0 0 0"/>
+  <joint name="gripper_joint1" type="prismatic">
+    <parent link="arm6_link"/>
+    <child link="gripper_left"/>
+    <origin rpy="0 0 0" xyz="0 0.09 0.05"/>
+    <axis xyz="0 1 0"/>
+    <limit lower="-0.08" upper="0" effort="100" velocity="0.1"/>
+  </joint>
+  <joint name="gripper_joint2" type="prismatic">
+    <parent link="arm6_link"/>
+    <child link="gripper_right"/>
+    <origin rpy="0 0 0" xyz="0 -0.09 0.05"/>
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