Commit message: Add files via upload

File: urdf/arm_old.xacro (robot description, xacro)
@@ -1,5 +1,35 @@
 <?xml version="1.0"?>
-<robot name="arm_robot">
-  <!-- Base of the arm(sliding rack)-->
+<robot name="arm_robot" xmlns:xacro="http://www.ros.org/wiki/xacro">
+  <!-- Properties -->
+  <xacro:property name="density" value="2700"/>  <!-- Density in kg/m^3 -->
+  <!-- Macro for calculating inertia for a box -->
+  <xacro:macro name="inertia_box" params="mass x y z">
+    <inertial>
+      <mass value="${mass}"/>
+      <origin rpy="0 0 0" xyz="0 0 0"/>
+      <inertia
+        ixx="${mass * (y*y + z*z) / 12.0}"
+        iyy="${mass * (x*x + z*z) / 12.0}"
+        izz="${mass * (x*x + y*y) / 12.0}"
+        ixy="0.0"
+        ixz="0.0"
+        iyz="0.0" />
+    </inertial>
+  </xacro:macro>
+  <!-- Macro for calculating inertia for a cylinder -->
+  <xacro:macro name="inertia_cylinder" params="mass radius length">
+    <inertial>
+      <mass value="${mass}"/>
+      <origin rpy="0 0 0" xyz="0 0 0"/>
+      <inertia
+        ixx="${mass * (3*radius*radius + length*length) / 12.0}"
+        iyy="${mass * (3*radius*radius + length*length) / 12.0}"
+        izz="${mass * radius*radius / 2.0}"
+        ixy="0.0"
+        ixz="0.0"
+        iyz="0.0" />
+    </inertial>
+  </xacro:macro>
+  <!-- Base Link -->
   <link name="base_link">
     <visual>
@@ -8,7 +38,4 @@
         <box size="0.2 1 0.1"/>
       </geometry>
-      <material name="blue">
-        <color rgba="0 0 1 1"/>
-      </material>
     </visual>
     <collision>
@@ -18,6 +45,7 @@
       </geometry>
     </collision>
-  </link>
-  <!-- Joint from Base to First link -->
+    <xacro:inertia_box mass="${density * 0.2 * 1 * 0.1}" x="0.2" y="1" z="0.1"/>
+  </link>
+  <!-- Prismatic Joint -->
   <joint name="arm1_p_joint" type="prismatic">
     <parent link="base_link"/>
@@ -25,5 +53,5 @@
     <origin rpy="0 0 0" xyz="0 0 0.1"/>
     <axis xyz="0 1 0"/>
-    <limit lower="-0.4" upper="0.4" effort="100" velocity="0.1"/>
+    <limit lower="-0.4" upper="0.4" effort="50" velocity="0.2"/>
   </joint>
   <!-- First Prismatic Link -->
@@ -32,18 +60,16 @@
       <origin rpy="0 0 0" xyz="0 0 0"/>
       <geometry>
-        <cylinder length="0.1" radius="0.1"/>
-      </geometry>
-      <material name="red">
-        <color rgba="1 0 0 1"/>
-      </material>
-    </visual>
-    <collision>
-      <origin rpy="0 0 0" xyz="0 0 0"/>
-      <geometry>
-        <cylinder length="0.1" radius="0.1"/>
-      </geometry>
-    </collision>
-  </link>
-  <!-- Joint from First prismatic to revolute link -->
+        <cylinder radius="0.1" length="0.1"/>
+      </geometry>
+    </visual>
+    <collision>
+      <origin rpy="0 0 0" xyz="0 0 0"/>
+      <geometry>
+        <cylinder radius="0.1" length="0.1"/>
+      </geometry>
+    </collision>
+    <xacro:inertia_cylinder mass="${density * 3.14 * 0.1 * 0.1 * 0.1}" radius="0.1" length="0.1"/>
+  </link>
+  <!-- Revolute Joint -->
   <joint name="arm1_r_joint" type="revolute">
     <parent link="arm1_p_link"/>
@@ -51,5 +77,5 @@
     <origin rpy="0 0 0" xyz="0 0 0.1"/>
     <axis xyz="0 0 1"/>
-    <limit lower="-1.55" upper="1.55" effort="100" velocity="0.1"/>
+    <limit lower="-3.14" upper="3.14" effort="50" velocity="1.0"/>
   </joint>
   <!-- First Revolute Link -->
@@ -58,24 +84,22 @@
       <origin rpy="0 0 0" xyz="0 0 0"/>
       <geometry>
-        <cylinder length="0.1" radius="0.1"/>
-      </geometry>
-      <material name="red">
-        <color rgba="1 0 0 1"/>
-      </material>
-    </visual>
-    <collision>
-      <origin rpy="0 0 0" xyz="0 0 0"/>
-      <geometry>
-        <cylinder length="0.1" radius="0.1"/>
-      </geometry>
-    </collision>
-  </link>
-  <!-- Joint from First revolute to arm2_link -->
+        <cylinder radius="0.1" length="0.1"/>
+      </geometry>
+    </visual>
+    <collision>
+      <origin rpy="0 0 0" xyz="0 0 0"/>
+      <geometry>
+        <cylinder radius="0.1" length="0.1"/>
+      </geometry>
+    </collision>
+    <xacro:inertia_cylinder mass="${density * 3.14 * 0.1 * 0.1 * 0.1}" radius="0.1" length="0.1"/>
+  </link>
+  <!-- Revolute Joint -->
   <joint name="arm2_joint" type="revolute">
     <parent link="arm1_r_link"/>
     <child link="arm2_link"/>
-    <origin rpy="0 0 0" xyz="0 -0.2 -0"/>
+    <origin rpy="0 0 0" xyz="0 -0.2 0"/>
     <axis xyz="0 1 0"/>
-    <limit lower="-1.68" upper="2.01" effort="100" velocity="0.1"/>
+    <limit lower="-3.14" upper="3.14" effort="50" velocity="1.0"/>
   </joint>
   <!-- Second Link -->
@@ -86,16 +110,10 @@
         <box size="0.2 0.2 0.1"/>
       </geometry>
-      <material name="red">
-        <color rgba="1 0 0 1"/>
-      </material>
-    </visual>
-    <visual>
-      <origin rpy="0 0 0" xyz="0 0 0.3"/>
-      <geometry>
-        <cylinder length="0.5" radius="0.1"/>
-      </geometry>
-      <material name="yellow">
-        <color rgba="1 1 0 1"/>
-      </material>
+    </visual>
+    <visual>
+      <origin rpy="0 0 0" xyz="0 0 0.3"/>
+      <geometry>
+        <cylinder radius="0.1" length="0.5"/>
+      </geometry>
     </visual>
     <visual>
@@ -104,18 +122,15 @@
         <box size="0.2 0.2 0.1"/>
       </geometry>
-      <material name="red">
-        <color rgba="1 0 0 1"/>
-      </material>
-    </visual>
-    <collision>
-      <origin rpy="0 0 0" xyz="0 0 0"/>
-      <geometry>
-        <box size="0.2 0.2 0.1"/>
-      </geometry>
-    </collision>
-    <collision>
-      <origin rpy="0 0 0" xyz="0 0 0.3"/>
-      <geometry>
-        <cylinder length="0.5" radius="0.1"/>
+    </visual>
+    <collision>
+      <origin rpy="0 0 0" xyz="0 0 0"/>
+      <geometry>
+        <box size="0.2 0.2 0.1"/>
+      </geometry>
+    </collision>
+    <collision>
+      <origin rpy="0 0 0" xyz="0 0 0.3"/>
+      <geometry>
+        <cylinder radius="0.1" length="0.5"/>
       </geometry>
     </collision>
@@ -126,6 +141,7 @@
       </geometry>
     </collision>
-  </link>
-  <!-- Joint from arm2_link to arm3_link -->
+    <xacro:inertia_box mass="${density * 0.2 * 0.2 * 0.1}" x="0.2" y="0.2" z="0.1"/>
+  </link>
+  <!-- Revolute Joint -->
   <joint name="arm3_joint" type="revolute">
     <parent link="arm2_link"/>
@@ -133,5 +149,5 @@
     <origin rpy="0 0 0" xyz="0 0.2 0.6"/>
     <axis xyz="0 1 0"/>
-    <limit lower="-2.80" upper="2.80" effort="100" velocity="0.1"/>
+    <limit lower="-3.14" upper="3.14" effort="50" velocity="1.0"/>
   </joint>
   <!-- Third Link -->
@@ -142,31 +158,26 @@
         <box size="0.2 0.2 0.1"/>
       </geometry>
-      <material name="red">
-        <color rgba="1 0 0 1"/>
-      </material>
-    </visual>
-    <visual>
-      <origin rpy="0 0 0" xyz="0 0 0.3"/>
-      <geometry>
-        <cylinder length="0.5" radius="0.1"/>
-      </geometry>
-      <material name="yellow">
-        <color rgba="1 1 0 1"/>
-      </material>
-    </visual>
-    <collision>
-      <origin rpy="0 0 0" xyz="0 0 0"/>
-      <geometry>
-        <box size="0.2 0.2 0.1"/>
-      </geometry>
-    </collision>
-    <collision>
-      <origin rpy="0 0 0" xyz="0 0 0.3"/>
-      <geometry>
-        <cylinder length="0.5" radius="0.1"/>
-      </geometry>
-    </collision>
-  </link>
-  <!-- Joint from arm3_link to arm4_link -->
+    </visual>
+    <visual>
+      <origin rpy="0 0 0" xyz="0 0 0.3"/>
+      <geometry>
+        <cylinder radius="0.1" length="0.5"/>
+      </geometry>
+    </visual>
+    <collision>
+      <origin rpy="0 0 0" xyz="0 0 0"/>
+      <geometry>
+        <box size="0.2 0.2 0.1"/>
+      </geometry>
+    </collision>
+    <collision>
+      <origin rpy="0 0 0" xyz="0 0 0.3"/>
+      <geometry>
+        <cylinder radius="0.1" length="0.5"/>
+      </geometry>
+    </collision>
+    <xacro:inertia_box mass="${density * 0.2 * 0.2 * 0.1}" x="0.2" y="0.2" z="0.1"/>
+  </link>
+  <!-- Prismatic Joint -->
   <joint name="arm4_joint" type="prismatic">
     <parent link="arm3_link"/>
@@ -174,5 +185,5 @@
     <origin rpy="0 0 0" xyz="0 0 0.3"/>
     <axis xyz="0 0 1"/>
-    <limit lower="0" upper="0.5" effort="100" velocity="0.1"/>
+    <limit lower="0" upper="0.5" effort="50" velocity="0.2"/>
   </joint>
   <!-- Fourth Link -->
@@ -181,9 +192,6 @@
       <origin rpy="0 0 0" xyz="0 0 0"/>
       <geometry>
-        <cylinder length="0.5" radius="0.08"/>
-      </geometry>
-      <material name="green">
-        <color rgba="0 1 0 1"/>
-      </material>
+        <cylinder radius="0.08" length="0.5"/>
+      </geometry>
     </visual>
     <visual>
@@ -192,12 +200,9 @@
         <cylinder length="0.1" radius="0.1" />
       </geometry>
-      <material name="red">
-        <color rgba="1 0 0 1"/>
-      </material>
-    </visual>
-    <collision>
-      <origin rpy="0 0 0" xyz="0 0 0"/>
-      <geometry>
-        <cylinder length="0.5" radius="0.08"/>
+    </visual>
+    <collision>
+      <origin rpy="0 0 0" xyz="0 0 0"/>
+      <geometry>
+        <cylinder radius="0.08" length="0.5"/>
       </geometry>
     </collision>
@@ -208,111 +213,15 @@
       </geometry>
     </collision>
-  </link>
-  <!-- Joint from arm4_link to arm5_link -->
-  <joint name="arm5_joint" type="revolute">
+    <xacro:inertia_cylinder mass="${density * 3.14 * 0.08 * 0.08 * 0.5}" radius="0.08" length="0.5"/>
+  </link>
+  <!-- Fixed Joint for Tool -->
+  <joint name="tool_joint" type="fixed">
     <parent link="arm4_link"/>
-    <child link="arm5_link"/>
-    <origin rpy="0 0 0" xyz="0 0 0.36"/>
-    <axis xyz="0 0 1"/>
-    <limit lower="-2.80" upper="2.80" effort="100" velocity="0.1"/>
-  </joint>
-  <!-- Fifth Link (base gripper) -->
-  <link name="arm5_link">
-    <!-- Circle base to revolute -->
-    <visual>
-      <origin rpy="0 0 0" xyz="0 0 0"/>
-      <geometry>
-        <cylinder radius="0.1" length="0.02"/>
-      </geometry>
-      <material name="green">
-        <color rgba="0 1 0 1"/>
-      </material>
-    </visual>
-    <!-- A box sliding rack mechanism for the gripper -->
-    <visual>
-      <origin rpy="0 0 0" xyz="0 0 0.02"/>
-      <geometry>
-        <box size="0.02 0.2 0.02"/>
-      </geometry>
-      <material name="white">
-        <color rgba="1 1 1 1"/>
-      </material>
-    </visual>
-    <!-- Collisions -->
-    <collision>
-      <origin rpy="0 0 0" xyz="0 0 0"/>
-      <geometry>
-        <cylinder radius="0.1" length="0.02"/>
-      </geometry>
-    </collision>
-    <collision>
-      <origin rpy="0 0 0" xyz="0 0 0.02"/>
-      <geometry>
-        <box size="0.02 0.2 0.02"/>
-      </geometry>
-    </collision>
-  </link>
-  <!-- ###Gripper### -->
-  <!-- Gripper link left -->
-  <link name="gripper_link_left">
-    <visual>
-      <origin rpy="0 0 0" xyz="0 0 0"/>
-      <geometry>
-        <box size="0.02 0.02 0.1"/>
-      </geometry>
-      <material name="white">
-        <color rgba="1 1 1 1"/>
-      </material>
-    </visual>
-    <collision>
-      <origin rpy="0 0 0" xyz="0 0 0"/>
-      <geometry>
-        <box size="0.02 0.02 0.1"/>
-      </geometry>
-    </collision>
-  </link>
-  <!-- Joint from arm5_link to gripper_link_left -->
-  <joint name="gripper_joint1" type="prismatic">
-    <parent link="arm5_link"/>
-    <child link="gripper_link_left"/>
-    <origin rpy="0 0 0" xyz="0 0.09 0.08"/>
-    <axis xyz="0 1 0"/>
-    <limit lower="-0.08" upper="0" effort="100" velocity="0.1"/>
-  </joint>
-  <!-- Gripper link right -->
-  <link name="gripper_link_right">
-    <visual>
-      <origin rpy="0 0 0" xyz="0 0 0"/>
-      <geometry>
-        <box size="0.02 0.02 0.1"/>
-      </geometry>
-      <material name="white">
-        <color rgba="1 1 1 1"/>
-      </material>
-    </visual>
-    <collision>
-      <origin rpy="0 0 0" xyz="0 0 0"/>
-      <geometry>
-        <box size="0.02 0.02 0.1"/>
-      </geometry>
-    </collision>
-  </link>
-  <!-- Joint from arm5_link to gripper_link_right -->
-  <joint name="gripper_joint2" type="prismatic">
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
File: urdf/irwb.xacro (robot description, xacro)
@@ -1,262 +1,15 @@
 <?xml version="1.0"?>
-<!-- ########################################### -->
-<!-- Description of iRWB (intelegent Runway Bot) -->
-<!-- Made by Phufar                              -->
-<!-- Feb 2025                                    -->
-<!-- ########################################### -->
-<robot name="runway_bot" xmlns:xacro="http://www.ros.org/wiki/xacro">
+<robot name="irwb_full" xmlns:xacro="http://www.ros.org/wiki/xacro">
+  <!-- Include mobile base model -->
+  <xacro:include filename="$(find irwb_robot_pkg)/urdf/irwb_body.xacro"/>
+  <!-- Include arm model -->
   <xacro:include filename="$(find irwb_robot_pkg)/urdf/arm.xacro"/>
-  <!-- Body dimensions -->
-  <xacro:property name="body_link_x_dim" value="2"/>
-  <xacro:property name="body_link_y_dim" value="1"/>
-  <xacro:property name="body_link_z_dim" value="0.7"/>
-  <xacro:property name="body_inner_x" value="0.8"/>
-  <xacro:property name="body_inner_y" value="0.8"/>
-  <xacro:property name="body_inner_z" value="0.6"/>
-  <!-- Wheel dimensions -->
-  <xacro:property name="wheel_link_radius" value="0.2"/>
-  <xacro:property name="wheel_link_length" value="0.15"/>
-  <xacro:property name="wheel_link_z_location" value="-0.3"/>
-  <!-- Material density -->
-  <xacro:property name="body_density" value="2710"/>
-  <xacro:property name="wheel_density" value="1500"/>
-  <!-- Pi const -->
-  <xacro:property name="pi_const" value="3.141592652589"/>
-  <!-- Robot body and wheel mass -->
-  <xacro:property name="body_mass" value="${body_density * body_link_x_dim * body_link_y_dim * body_link_z_dim}"/>
-  <xacro:property name="wheel_mass" value="${
-   wheel_density * pi_const * wheel_link_radius * wheel_link_radius * wheel_link_length}"/>
-  <!-- Moment of inertia of the wheel -->
-  <xacro:property name="Iz_wheel" value="${0.5 * wheel_mass * wheel_link_radius * wheel_link_radius}"/>
-  <xacro:property name="I_wheel" value="${
-   (1.0/12.0) * wheel_mass * wheel_link_radius * wheel_link_radius + wheel_link_length * wheel_link_length}"/>
-  <!-- macro of the complete inertial section of wheel -->
-  <xacro:macro name="inertia_wheel">
-    <inertial>
-      <origin rpy="0 0 0" xyz="0 0 0"/>
-      <mass value="${wheel_mass}"/>
-      <inertia ixx="${I_wheel}" ixy="0.0" ixz="0.0" iyy="${I_wheel}" iyz="0.0" izz="${Iz_wheel}"/>
-    </inertial>
-  </xacro:macro>
-  <!-- Import saved gazebo settings next time we run -->
-  <xacro:include filename="$(find irwb_robot_pkg)/urdf/robot.gazebo"/>
-  <!--####################################-->
-  <!--# Define all Links and Joints here #-->
-  <!--####################################-->
-  <!-- Mandatory "dummy" link and joint -->
-  <link name="dummy"></link>
-  <joint name="dummy_joint" type="fixed">
-    <parent link="dummy"/>
-    <child link="body_link"/>
-  </joint>
-  <!--####################################-->
-  <!--# body_link with hole in the front #-->
-  <!--####################################-->
-  <link name="body_link">
-    <visual>
-      <origin rpy="0 0 0" xyz="${-1 * body_link_x_dim / 4} 0 0"/>
-      <geometry>
-        <box size="${body_link_x_dim / 2} ${body_link_y_dim} ${body_link_z_dim}"/>       <!-- Solid back part -->
-      </geometry>
-    </visual>
-    <visual>
-      <origin rpy="0 0 0" xyz="${(body_link_x_dim/2 - body_inner_x)/4.0} 0 0"/>       <!-- Shaded area 1 -->
-      <geometry>
-        <box size="0.1 ${body_inner_y} ${body_link_z_dim}"/>
-      </geometry>
-    </visual>
-    <visual>
-      <origin rpy="0 0 0" xyz="${(body_link_x_dim/2 - body_inner_x)/4 + 0.9} 0 0"/>  <!-- Shaded area 2 -->
-      <geometry>
-        <box size="0.1 ${body_inner_y} ${body_link_z_dim}"/>
-      </geometry>
-    </visual>
-    <visual>
-      <origin rpy="0 0 0" xyz="${body_link_x_dim / 4} ${(body_link_y_dim - 0.1)/ 2} 0"/>  <!-- Unshaded area 1 -->
-      <geometry>
-        <box size="${body_inner_x + 0.2} 0.1 ${body_link_z_dim}"/>
-      </geometry>
-    </visual>
-    <visual>
-      <origin rpy="0 0 0" xyz="${body_link_x_dim / 4} ${-1 * (body_link_y_dim - 0.1)/ 2} 0"/> <!-- Unshaded area 2 -->
-      <geometry>
-        <box size="${body_inner_x + 0.2} 0.1 ${body_link_z_dim}"/>
-      </geometry>
-    </visual>
-    <visual>
-      <origin rpy="0 0 0" xyz="${body_link_x_dim / 4} 0 ${-1 * (body_link_z_dim - 0.1)/2}"/> <!-- Base of hole -->
-      <geometry>
-        <box size="${body_inner_x} ${body_inner_y} 0.1"/>
-      </geometry>
-    </visual>
-    <collision>
-      <origin rpy="0 0 0" xyz="${-1 * body_link_x_dim / 4} 0 0"/>
-      <geometry>
-        <box size="${body_link_x_dim / 2} ${body_link_y_dim} ${body_link_z_dim}"/>
-      </geometry>
-    </collision>
-    <collision>
-      <origin rpy="0 0 0" xyz="${(body_link_x_dim/2 - body_inner_x)/4.0} 0 0"/>
-      <geometry>
-        <box size="0.1 ${body_inner_y} ${body_link_z_dim}"/>
-      </geometry>
-    </collision>
-    <collision>
-      <origin rpy="0 0 0" xyz="${(body_link_x_dim/2 - body_inner_x)/4 + 0.9} 0 0"/>
-      <geometry>
-        <box size="0.1 ${body_inner_y} ${body_link_z_dim}"/>
-      </geometry>
-    </collision>
-    <collision>
-      <origin rpy="0 0 0" xyz="${body_link_x_dim / 4} ${(body_link_y_dim - 0.1)/ 2} 0"/>
-      <geometry>
-        <box size="${body_inner_x + 0.2} 0.1 ${body_link_z_dim}"/>
-      </geometry>
-    </collision>
-    <collision>
-      <origin rpy="0 0 0" xyz="${body_link_x_dim / 4} ${-1 * (body_link_y_dim - 0.1)/ 2} 0"/>
-      <geometry>
-        <box size="${body_inner_x + 0.2} 0.1 ${body_link_z_dim}"/>
-      </geometry>
-    </collision>
-    <collision>
-      <origin rpy="0 0 0" xyz="${body_link_x_dim / 4} 0 ${-1 * (body_link_z_dim - 0.1)/2}"/>
-      <geometry>
-        <box size="${body_inner_x} ${body_inner_y} 0.1"/>
-      </geometry>
-    </collision>
-    <inertial>
-      <origin rpy="0 0 0" xyz="0 0 0"/>
-      <mass value="${body_mass}"/>
-      <inertia
-      ixx="${(1.0/12.0) * body_mass * (body_link_y_dim * body_link_y_dim + body_link_z_dim * body_link_z_dim)}"
-      ixy="0"
-      ixz="0"
-      iyy="${(1.0/12.0) * body_mass * (body_link_x_dim * body_link_x_dim + body_link_z_dim * body_link_z_dim)}"
-      iyz="0"
-      izz="${(1.0/12.0) * body_mass * (body_link_x_dim * body_link_x_dim + body_link_y_dim * body_link_y_dim)}"
-      />
-    </inertial>
-  </link>
-  <!--####################################-->
-  <!--#         end of body_link         #-->
-  <!--####################################-->
- <!--# Joint from iRWB to wheel 1 #-->
- <joint name="wheel1_joint" type="continuous">
-  <parent link="body_link"/>
-  <child link="wheel1_link"/>
-  <origin rpy="0 0 0" xyz="
-   ${-1 * (body_link_x_dim/2 - 1.2 * wheel_link_radius)}
-   ${-1 * (body_link_y_dim/2 + wheel_link_length/2)}
-   ${wheel_link_z_location}"/>
-  <axis xyz="0 1 0"/>
-  <limit effort="1000" velocity="1000"/>
-  <dynamics damping="1.0" friction="1.0"/>
- </joint>
-  <!--### back right wheel1 ###-->
-  <link name="wheel1_link">
-    <visual>
-      <origin rpy="1.5708 0 0" xyz="0 0 0"/>
-      <geometry>
-        <cylinder length="${wheel_link_length}" radius="${wheel_link_radius}"/>
-      </geometry>
-    </visual>
-    <collision>
-      <origin rpy="1.5708 0 0" xyz="0 0 0"/>
-      <geometry>
-        <cylinder length="${wheel_link_length}" radius="${wheel_link_radius}"/>
-      </geometry>
-    </collision>
-    <xacro:inertia_wheel/>
-  </link>
-  <!--# Joint from iRWB to wheel 2 #-->
-  <joint name="wheel2_joint" type="continuous">
-    <parent link="body_link"/>
-    <child link="wheel2_link"/>
-    <origin rpy="0 0 0" xyz="
-     ${-1 * (body_link_x_dim/2 - 1.2 * wheel_link_radius)}
-     ${1 * (body_link_y_dim/2 + wheel_link_length/2)}
-     ${wheel_link_z_location}"/>
-    <axis xyz="0 1 0"/>
-    <limit effort="1000" velocity="1000"/>
-    <dynamics damping="1.0" friction="1.0"/>
-  </joint>
-  <!--### back left wheel2 ###-->
-  <link name="wheel2_link">
-    <visual>
-      <origin rpy="1.5708 0 0" xyz="0 0 0"/>
-      <geometry>
-        <cylinder length="${wheel_link_length}" radius="${wheel_link_radius}"/>
-      </geometry>
-    </visual>
-    <collision>
-      <origin rpy="1.5708 0 0" xyz="0 0 0"/>
-      <geometry>
-        <cylinder length="${wheel_link_length}" radius="${wheel_link_radius}"/>
-      </geometry>
-    </collision>
-    <xacro:inertia_wheel/>
-  </link>
-   <!--# Joint from iRWB to wheel 3 #-->
-  <joint name="wheel3_joint" type="continuous">
-    <parent link="body_link"/>
-    <child link="wheel3_link"/>
-    <origin rpy="0 0 0" xyz="
-     ${1 * (body_link_x_dim/2 - 1.2 * wheel_link_radius)}
-     ${-1 * (body_link_y_dim/2 + wheel_link_length/2)}
-     ${wheel_link_z_location}"/>
-    <axis xyz="0 1 0"/>
-    <limit effort="1000" velocity="1000"/>
-    <dynamics damping="1.0" friction="1.0"/>
-  </joint>
-  <!--### front right wheel3 ###-->
-  <link name="wheel3_link">
-    <visual>
-      <origin rpy="1.5708 0 0" xyz="0 0 0"/>
-      <geometry>
-        <cylinder length="${wheel_link_length}" radius="${wheel_link_radius}"/>
-      </geometry>
-    </visual>
-    <collision>
-      <origin rpy="1.5708 0 0" xyz="0 0 0"/>
-      <geometry>
-        <cylinder length="${wheel_link_length}" radius="${wheel_link_radius}"/>
-      </geometry>
-    </collision>
-    <xacro:inertia_wheel/>
-  </link>
-   <!--# Joint from iRWB to wheel 4 #-->
-  <joint name="wheel4_joint" type="continuous">
-    <parent link="body_link"/>
-    <child link="wheel4_link"/>
-    <origin rpy="0 0 0" xyz="
-     ${1 * (body_link_x_dim/2 - 1.2 * wheel_link_radius)}
-     ${1 * (body_link_y_dim/2 + wheel_link_length/2)}
-     ${wheel_link_z_location}"/>
-    <axis xyz="0 1 0"/>
-    <limit effort="1000" velocity="1000"/>
-    <dynamics damping="1.0" friction="1.0"/>
-  </joint>
-  <!--### front left wheel4 ###-->
-  <link name="wheel4_link">
-    <visual>
-      <origin rpy="1.5708 0 0" xyz="0 0 0"/>
-      <geometry>
-        <cylinder length="${wheel_link_length}" radius="${wheel_link_radius}"/>
-      </geometry>
-    </visual>
-    <collision>
-      <origin rpy="1.5708 0 0" xyz="0 0 0"/>
-      <geometry>
-        <cylinder length="${wheel_link_length}" radius="${wheel_link_radius}"/>
-      </geometry>
-    </collision>
-    <xacro:inertia_wheel/>
-  </link>
-  <!-- Fixed Joint from arm to body -->
+  <!-- Mount the arm onto the base with a fixed joint.
+       Adjust the xyz values so that the arm is mounted at the proper height.
+       In this example, we attach the arm’s base_link to the body_link. -->
   <joint name="arm_mount_joint" type="fixed">
     <parent link="body_link"/>
     <child link="base_link"/>
-    <origin rpy="0 0 0" xyz="0 0 0.4"/>
+    <origin xyz="0 0 0.4" rpy="0 0 0"/>
   </joint>
 </robot>
